File: hardware/opera-mitm/board/s660-pdb-mitm.kicad_pcb (KiCad board)
At the start: 2 copper layers, 90 x 90 mm, 89 parts, among them J1 JST B7B-XH-A, J101 MC 1,5/4-G-5.08, J102 MC 1,5/2-G-5.08, J103 Pi link 2x5, J104 ISP 2x3 DNP, J2 JST B3B-XH-A, K1 G6K-2F-Y 5VDC, K101 G2RL-1A DC12, Q1 2N7002, Q102 MMBT2222A, Q103 2N7002, Q2 2N7002, Q3 2N7002, Q4 2N7002, Q5 2N7002, SW101 TS-1187A-B-A-B, SW2 TS-1187A-B-A-B, U1 Raspberry Pi Pico 2 W, U101 ATtiny85-20SU, U102 LM2936MPX-3.3, U103 EL817S

Commit message: Buddy board rev B: Phoenix MC harness header, Pico socketed (DNP), labelled back silkscreen
J1 (car-harness OPERA lines) is now a Phoenix MC 1,5/7-G-5.08 pluggable header on the top
edge between J102 and J101, replacing the mid-board JST XH: the harness pigtail gets ferrules
and a MC 1,5/7-ST-5.08 plug, matching the power terminals. Same pin order (1 TXp ... 7 GND).
U102 (LM2936) with C105/C107 moved into the pocket the JST left, beside K1; its 12V feed,
3V3_AON output and the six J1 nets re-routed, RLY_COIL re-routed to clear the LDO pad.

U1 (Pico 2 W) is marked do-not-populate: the owner supplies the module and the board gets
two 1x20 female headers, listed in the hand-fit BOM. Mounting holes set to 4.0 mm from the
sides and 6.1 mm from top/bottom to match the TOFU.

Silkscreen: back-side labels name every wire at J101 (Constant/ACC/IG2/Ground, Honda option
coupler), J1 (panel pins, panel/HU side) and J102 (12V OUT/GND), plus a J103-to-Pi-GPIO
table; front carries the board title and LED legends.

Checks: DRC 0/0/0 with the Power12V (0.3 mm) and Supply net classes in force, schematic
parity 0, schematic-to-board netlist identical on all 262 pads, one GND net, ERC only the
known Pico-symbol GND/AGND artefact.

fab/rev-B replaces fab/rev-A (never ordered): Gerbers + drills (186 PTH = 90 THT pads + 96
vias, 4 NPTH), JLCPCB SMT BOM/CPL (72 parts, 27 line items, all with LCSC numbers), hand-fit
list, README with the upload steps and the mandatory placement-preview note.

COMBINED.md/DESIGN.md record the J1 change and the corrected Phoenix order number (1836231).

Co-Authored-By: Claude Fable 5.1 <noreply@anthropic.com>
Parts:
- J1: value JST B7B-XH-A -> MC 1,5/7-G-5.08; footprint Connector_JST:JST_XH_B7B-XH-A_1x07_P2.50mm_Vertical -> Connector_Phoenix_MC_HighVoltage:PhoenixContact_MC_1,5_7-G-5.08_1x07_P5.08mm_Horizontal
- moved J1 48.8 mm to (67.6, 16.8), turned to 180 degrees
- moved C107 29.0 mm to (40.0, 46.6)
- moved U102 28.4 mm to (32.5, 44.4)
- moved C105 22.3 mm to (27.0, 41.5), turned to 0 degrees
- moved J2 9.56 mm to (60.9, 56.6)
- moved LED103 0.61 mm to (88.6, 94.1)
- moved R116 0.60 mm to (88.7, 97.8)
- moved R114 0.15 mm to (76.2, 97.8)
- moved R115 0.11 mm to (82.2, 97.8)
- moved J102 0.06 mm to (28.3, 16.8)
- moved J101 0.05 mm to (91.5, 16.8)
Routing:
- net /TXp: track 25.5 -> 106.8 mm, vias 3 -> 2
- net /CONT: track 29.9 -> 78.8 mm, vias 2 -> 5
- net /RX: track 29.9 -> 67.0 mm, vias 2 -> 5
- net /PWp: track 38.7 -> 75.7 mm, vias 3 -> 4
- net /TXh: track 39.3 -> 75.8 mm, vias 3 -> 4
- net /PWh: track 58.3 -> 82.8 mm, vias 1 -> 3
- net /RUN_PG: track 4.54 -> 10.7 mm
- net /+3V3_AON: track 78.0 -> 73.4 mm
- net /12V_IN: track 162.2 -> 165.2 mm, vias 0 -> 2
- net /12V_SW: track 188.6 -> 187.6 mm
- net /RLY_COIL: track 53.0 -> 53.1 mm, vias 0 -> 2
Other:
- board text added: "1 GND 3 HALT G26 5 FAN G18 7 MOSI G5 9 RST G13"
- board text added: "12V OUT"
- board text added: "Accessory (ACC Red)"
- board text added: "Atiny85 HEARTBEAT"
- board text added: "Constant (+B Yellow)"
- board text added: "G17 IGN 2 G27 SHDN 4 G23 TACH 6 G6 MISO 8 GND 10"
- board text added: "GND"
- board text added: "Ground (Chassis)"
- board text added: "HARNESS"
- board text added: "Ignition (IG2 Red/Pink)"
- board text added: "MIDSHIP AMUSEMENT"
- board text added: "OPTION COUPLER"
- board text added: "POWER TEST"
- board text added: "Pin 1 HU Side"
- board text added: "Pin 1 Panel Side"
- board text added: "Pin 12"
- board text added: "Pin 2"
- board text added: "Pin 3 HU Side"
- board text added: "Pin 3 Panel Side"
- board text added: "Pin 8 GND"
- board text added: "RASPBERRY PI GPIO"
- board text added: "RELAY ON"
- board text added: "Raspberry Pi Pico 2 W"
- board text added: "S660 CarPlay Buddy Board Rev. B"
- board text added: "TOFU BOARD"
- board text added: "USB"
- board text added: "https://github.com/CLedebur/react-carplay-s660"

Commit message: Buddy board rev B: silkscreen corrections, J1 order number, final fab export
Silkscreen: J1 ground pin now "Pin 9 GND" (panel pin 9, per BUILD_NOTES §30.1), J102 terminal
"12V OUT" (it is the relay-switched feed to the TOFU, not an input), "ATtiny85 HEARTBEAT"
spelling, GPIO table last row "GND 10". "Option Coupler" is the Honda connector name and stays.

J1 MPN corrected to the KiCad library's Phoenix order number, MC 1,5/7-G-5.08 (1836231),
on both schematic and board (parity 0).

fab/rev-B regenerated from the saved board: DRC 0/0/0, parity 0, 186 PTH = 90 pads + 96 vias,
4 NPTH, SMT BOM/CPL 72 parts in 27 line items with LCSC numbers, hand-fit list with the Pico
sockets and the J1 mating plug.

Co-Authored-By: Claude Fable 5.1 <noreply@anthropic.com>
Other:
- board text added: "ATtiny85 HEARTBEAT"
- board text added: "Pin 9 GND"
- board text removed: "Atiny85 HEARTBEAT"
- board text removed: "Pin 8 GND"
Changed lines of the file:
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@@
 			)
 		)
-		(property "MPN" "MC 1,5/7-G-5.08 (1836312)"
+		(property "MPN" "MC 1,5/7-G-5.08 (1836231)"
 			(at 0 0 180)
 			(unlocked yes)
@@
 		)
 	)
-	(gr_text "Atiny85\nHEARTBEAT"
+	(gr_text "ATtiny85\nHEARTBEAT"
 		(at 88.93 100.07 0)
 		(layer "F.SilkS")
@@
 		)
 	)
-	(gr_text "Pin 8 GND"
+	(gr_text "Pin 9 GND"
 		(at 37.76 18.79 90)
 		(layer "B.SilkS")
